Commit message: AMCL lab updates -per grader recommendations

File: chase/src/my_robot/urdf/my_robot.xacro (robot description, xacro)
@@ -147,5 +147,5 @@
         <origin xyz="0 0 0" rpy=" 0 0 0" />
         <geometry>
-            <mesh filename="package://my_robot/meshes/hokuyo.dae" />
+            <mesh filename="$(find my_robot)/meshes/hokuyo.dae" />
         </geometry>
     </visual>
